File: eagle/Projects/Sij/Sij.brd (EAGLE design)
At the start: 111.4 x 186.7 mm, 59 parts, among them U1 ATMEGA2560AU, U2 BQ76925_PW_20, U3 LM1085_KTT_3, U4 LM7805

Commit message: joué avec le schematic et la commande digikey
Parts:
- removed JUMP_3_CELL, JUMP_4_CELL, JUMP_5_CELL, JUMP_PWR_BAT, JUMP_PWR_PROG: (no value), SparkFun-Connectors:1X02
- added CRESET, C_DECOUPLING1, C_DECOUPLING2, C_DECOUPLING3, C_DECOUPLING4: 0.1uF, SparkFun-Capacitors:0603-CAP
- added C_AVCC: 0.1u, SparkFun-Capacitors:0603-CAP
- added D1, D2: 1N4004, diode:DO41-10
- added D_POWER_SEL: (no value), SparkFun-DiscreteSemi:SMA-DIODE_ALT
- added JP1, JP2, JP3: (no value), SparkFun-Retired:1X02
- added L1: 10uH, SparkFun-Passives:0805
- added LED1, LED2, LED3, LED4, LED5, LED6, LED7: (no value), led:CHIPLED_0805
- added Q_POWER_SEL1: MOSFET-PCHANNEL, SparkFun-DiscreteSemi:SOT23-3
- added Q_POWER_SEL2: MOSFET-NCHANNELAO3404A, SparkFun-DiscreteSemi:SOT23-3
- added RESET_SWITCH: SWITCH-MOMENTARY-2PTH, SparkFun-Electromechanical:TACTILE-PTH
- added RLED1, RLED3, RLED4, RLED5, RLED6, RLED7: 56, resistor:R0603
- added RLED2: 316, resistor:R0603
- added RSCL, RSDA: 2K, resistor:R0603
- added RSS: 1K, resistor:R0603
- added R_PULL_DOWN_POWER_SEL, R_PULL_UP_POWER_SEL: 10K, resistor:R0603
- added R_RESET_SWITCH: 363, resistor:R0603
- added S1: (no value), SparkFun-Electromechanical:SWITCH-SPDT
- added U5: TC7SU04F, SparkFun-DigitalIC:SOT23-5
- renumbered C1 to C_CRYSTAL_1, C2 to C_CRYSTAL_2, R1 to R_1085, Y1 to CRYSTAL
Connections:
- removed net AGND: U1.99
- removed net AVCC: U1.100
- new net N$14: BAT+.P$1, ESC1+.IN, ESC2+.IN, ESC3+.IN, ESC4+.IN, RLED2.1, S1.2, S1.3
- new net N$34: RESET_SWITCH.1, R_RESET_SWITCH.2
- new net N$37: Q_POWER_SEL1.1, Q_POWER_SEL2.3, R_PULL_UP_POWER_SEL.1
- new net N$38: LED3.A, RLED3.2
- new net N$39: LED6.A, RLED6.2
- new net N$4: CIN_7805.1, Q_POWER_SEL1.2, U4.1
- new net N$41: LED7.A, RLED7.2
- new net N$42: RSS.1, U1.19
- new net N$5: C_AVCC.1, L1.2, U1.100
- new net RLED2: LED2.A, RLED2.2
- new net SCL: RSCL.2, U1.43, U2.19
- new net SDA: RSDA.2, U1.44, U2.18
- new net VCC1: RLED4.1, U1.59
- new net VCC2: RLED5.1, U1.58
- new net VCC3: RLED6.1
- new net VCC4: RLED7.1
- new net V_USB: D_POWER_SEL.A, ICSP.2, RLED3.1, U5.2
- net GND: now also CRESET.2, C_AVCC.2, C_DECOUPLING1.2, C_DECOUPLING2.2, C_DECOUPLING3.2, C_DECOUPLING4.2, D1.A, LED4.C, LED5.C, LED6.C, LED7.C, Q_POWER_SEL2.2, RESET_SWITCH.3, RSS.2, R_PULL_DOWN_POWER_SEL.1, U1.99, U5.3; no longer U1.19
- net N$13: now also Q_POWER_SEL2.1, R_PULL_DOWN_POWER_SEL.2, U5.4; no longer COUT_7805.1, JUMP_PWR_BAT.2, U4.3
- net N$19: now also LED4.A, RLED4.2; no longer U2.18
- net N$20: now also U1.79
- net N$21: now also U1.88
- net N$22: now also U1.87
- net N$24: now also U1.86
- net N$25: now also LED5.A, RLED5.2; no longer U2.19
- net N$28: now also JP3.1; no longer JUMP_3_CELL.1
- net N$29: now also JP2.1, JP3.2; no longer JUMP_3_CELL.2, JUMP_4_CELL.1
- net N$3: now also CRESET.1, D1.C, D2.A, R_RESET_SWITCH.1
- net N$30: now also JP1.1, JP2.2; no longer JUMP_4_CELL.2, JUMP_5_CELL.1
- net N$35: now also LED1.A, RLED1.2; no longer ICSP.2, JUMP_PWR_PROG.1
- net VCC: now also COUT_7805.1, C_DECOUPLING1.1, C_DECOUPLING2.1, C_DECOUPLING3.1, C_DECOUPLING4.1, D2.C, D_POWER_SEL.C, L1.1, RLED1.1, RSCL.1, RSDA.1, U4.3, U5.5; no longer JUMP_PWR_BAT.1, JUMP_PWR_PROG.2
- net V_BATT: now also JP1.2, Q_POWER_SEL1.3, R_PULL_UP_POWER_SEL.2, S1.1; no longer BAT+.P$1, CIN_7805.1, ESC1+.IN, ESC2+.IN, ESC3+.IN, ESC4+.IN, JUMP_5_CELL.2, U4.1

Commit message: fini le schematic préliminaire+bibliothèques de partie+documentation
Parts:
- removed S1: (no value), SparkFun-Electromechanical:SWITCH-SPDT
- added J_RECEIVER_GND, J_RECEIVER_SIG, J_RECEIVER_VCC: (no value), SparkFun-Connectors:1X07
- added LED10, LED11, LED8, LED9: (no value), led:CHIPLED_0805
- added RLED10, RLED11, RLED8, RLED9: 91, resistor:R0603
- added SG1: BUZZERPTH, SparkFun-Electromechanical:BUZZER-12MM
- added U$2: M06_IMU, custom_parts:1X06_LONGPADS
- added U$3: SWITCH_3_PIN, custom_parts:SWITCH-SPDT_KIT
- CRYSTAL: value (none) -> 16MHz
- D_POWER_SEL: value (none) -> CDBA320L
- ESC1_PWM, ESC3_PWM, ESC4_PWM: value (none) -> 640455 TE connectivity
- ICSP: device SparkFun-Connectors:2X5-SHROUDED -> SparkFun-Connectors:2X5_NOSILK
Connections:
- removed net VCC1: RLED4.1, U1.59
- removed net VCC2: RLED5.1, U1.58
- removed net VCC3: RLED6.1
- removed net VCC4: RLED7.1
- new net CH1: J_RECEIVER_SIG.1, U1.63
- new net CH2: J_RECEIVER_SIG.2, U1.64
- new net CH3: J_RECEIVER_SIG.3, U1.65
- new net CH4: J_RECEIVER_SIG.4, U1.66
- new net CH5: J_RECEIVER_SIG.5, U1.67
- new net CH6: J_RECEIVER_SIG.6, U1.68
- new net INT_IMU: U$2.2, U1.45
- new net N$43: LED8.A, RLED8.2
- new net N$44: LED9.A, RLED9.2
- new net N$45: LED10.A, RLED10.2
- new net N$46: LED11.A, RLED11.2
- new net N$47: RLED4.1, U1.60
- new net N$48: RLED5.1, U1.59
- new net N$49: RLED6.1, U1.58
- new net N$50: RLED7.1, U1.57
- new net N$51: RLED8.1, U1.56
- new net N$52: RLED9.1, U1.55
- new net N$53: RLED10.1, U1.54
- new net N$54: RLED11.1, U1.53
- new net N$55: SG1.-, U1.40
- net GND: now also J_RECEIVER_GND.1, J_RECEIVER_GND.2, J_RECEIVER_GND.3, J_RECEIVER_GND.4, J_RECEIVER_GND.5, J_RECEIVER_GND.6, LED10.C, LED11.C, LED8.C, LED9.C, SG1.+, U$2.1, U$2.5
- net N$14: now also U$3.2, U$3.3; no longer S1.2, S1.3
- net SCL: now also U$2.3
- net SDA: now also U$2.4
- net VCC: now also J_RECEIVER_VCC.1, J_RECEIVER_VCC.2, J_RECEIVER_VCC.3, J_RECEIVER_VCC.4, J_RECEIVER_VCC.5, J_RECEIVER_VCC.6, U$2.6
- net V_BATT: now also U$3.1; no longer S1.1

Commit message: listes matériel
Parts:
- CSENSE: device rcl:C0805 -> SparkFun-Passives:0603-CAP
Changed lines of the file:
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@@
 <attribute name="PROD_ID" value="CAP-00868" x="-8.89" y="-186.69" size="1.778" layer="27" display="off"/>
 </element>
-<element name="CSENSE" library="rcl" package="C0805" value="0.1u" x="-8.89" y="-193.04"/>
+<element name="CSENSE" library="SparkFun-Passives" package="0603-CAP" value="0.1u" x="-8.89" y="-193.04"/>
 <element name="RSENSEN" library="resistor" package="R0603" value="1K" x="-8.89" y="-199.39"/>
 <element name="RSENSEP" library="resistor" package="R0603" value="1K" x="-8.89" y="-205.74"/>
@@
 <contactref element="CSENSE" pad="1"/>
 <contactref element="U2" pad="11"/>
-<wire x1="-9.84" y1="-193.04" x2="-8.04" y2="-199.39" width="0" layer="19" extent="1-1"/>
-<wire x1="7.8994" y1="-8.005" x2="-9.84" y2="-193.04" width="0" layer="19" extent="1-1"/>
+<wire x1="-9.74" y1="-193.04" x2="-8.04" y2="-199.39" width="0" layer="19" extent="1-1"/>
+<wire x1="7.8994" y1="-8.005" x2="-9.74" y2="-193.04" width="0" layer="19" extent="1-1"/>
 </signal>
 <signal name="N$16">
@@
 <contactref element="CSENSE" pad="2"/>
 <contactref element="U2" pad="12"/>
-<wire x1="-7.94" y1="-193.04" x2="-8.04" y2="-205.74" width="0" layer="19" extent="1-1"/>
-<wire x1="7.8994" y1="-7.355003125" x2="-7.94" y2="-193.04" width="0" layer="19" extent="1-1"/>
+<wire x1="-8.04" y1="-193.04" x2="-8.04" y2="-205.74" width="0" layer="19" extent="1-1"/>
+<wire x1="7.8994" y1="-7.355003125" x2="-8.04" y2="-193.04" width="0" layer="19" extent="1-1"/>
 </signal>
 <signal name="N$20">

Commit message: quelques ports ajoutés
Parts:
- added PORTA, PORTE, PORTF: (no value), SparkFun-Connectors:AVR_ICSP
- ICSP: device SparkFun-Connectors:2X5_NOSILK -> SparkFun-Connectors:AVR_ICSP
Connections:
- new net PA0: PORTA.1, U1.78
- new net PA1: PORTA.2, U1.77
- new net PA2: PORTA.3, U1.76
- new net PA3: PORTA.4, U1.75
- new net PA4: PORTA.5, U1.74
- new net PA5: PORTA.6, U1.73
- new net PA6: PORTA.7, U1.72
- new net PA7: PORTA.8, U1.71
- new net PE0: PORTE.1, U1.2
- new net PE1: PORTE.2, U1.3
- new net PE2: PORTE.3, U1.4
- new net PE3: PORTE.4, U1.5
- new net PE4: PORTE.5, U1.6
- new net PE5: PORTE.6, U1.7
- new net PE6: PORTE.7, U1.8
- new net PE7: PORTE.8, U1.9
- new net PF0: PORTF.1, U1.97
- new net PF1: PORTF.2, U1.96
- new net PF2: PORTF.3, U1.95
- new net PF3: PORTF.4, U1.94
- new net PF4: PORTF.5, U1.93
- new net PF5: PORTF.6, U1.92
- new net PF6: PORTF.7, U1.91
- new net PF7: PORTF.8, U1.90
- net GND: now also PORTA.9, PORTE.9, PORTF.9
- net VCC: now also PORTA.10, PORTE.10, PORTF.10
Changed lines of the file:
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@@
 </autorouter>
 <elements>
-<element name="ICSP" library="SparkFun-Connectors" package="2X5_NOSILK" value="" x="26.67" y="39.37" rot="R90"/>
+<element name="ICSP" library="SparkFun-Connectors" package="AVR_ICSP" value="" x="26.67" y="39.37" rot="R90"/>
 <element name="U1" library="SparkFun-DigitalIC" package="TQFP100" value="ATMEGA2560AU" x="52.07" y="39.37">
 <attribute name="PROD_ID" value="IC-10040" x="52.07" y="39.37" size="1.778" layer="27" display="off"/>
@@
 <element name="J_RECEIVER_GND" library="SparkFun-Connectors" package="1X07" value="" x="-125.73" y="-740.41"/>
 <element name="SG1" library="SparkFun-Electromechanical" package="BUZZER-12MM" value="BUZZERPTH" x="-120.65" y="-748.03"/>
+<element name="PORTA" library="SparkFun-Connectors" package="AVR_ICSP" value="" x="-130.81" y="-746.76"/>
+<element name="PORTE" library="SparkFun-Connectors" package="AVR_ICSP" value="" x="-137.16" y="-746.76"/>
+<element name="PORTF" library="SparkFun-Connectors" package="AVR_ICSP" value="" x="-143.51" y="-746.76"/>
 </elements>
 <signals>
@@
 <contactref element="J_RECEIVER_GND" pad="6"/>
 <contactref element="SG1" pad="+"/>
+<contactref element="PORTA" pad="9"/>
+<contactref element="PORTE" pad="9"/>
+<contactref element="PORTF" pad="9"/>
 <wire x1="-71.12" y1="-683.48" x2="-76.2" y2="-683.48" width="0" layer="19" extent="1-1"/>
 <wire x1="-76.2" y1="-672.05" x2="-76.2" y2="-683.48" width="0" layer="19" extent="1-1"/>
@@
 <wire x1="-125.73" y1="-740.41" x2="-123.19" y2="-740.41" width="0" layer="19" extent="1-1"/>
 <wire x1="-117.4" y1="-748.03" x2="-118.11" y2="-740.41" width="0" layer="19" extent="1-1"/>
+<wire x1="-132.08" y1="-751.84" x2="-125.73" y2="-740.41" width="0" layer="19" extent="1-1"/>
+<wire x1="-138.43" y1="-751.84" x2="-132.08" y2="-751.84" width="0" layer="19" extent="1-1"/>
+<wire x1="-144.78" y1="-751.84" x2="-138.43" y2="-751.84" width="0" layer="19" extent="1-1"/>
 <wire x1="-49.85" y1="-604.25" x2="-76.62" y2="-645.16" width="0" layer="19" extent="1-1"/>
 <wire x1="-46.04" y1="-603.2801" x2="-49.85" y2="-604.25" width="0" layer="19" extent="1-1"/>
@@
 <contactref element="J_RECEIVER_VCC" pad="5"/>
 <contactref element="J_RECEIVER_VCC" pad="6"/>
+<contactref element="PORTA" pad="10"/>
+<contactref element="PORTE" pad="10"/>
+<contactref element="PORTF" pad="10"/>
 <wire x1="-78.32" y1="-655.32" x2="-83.82" y2="-665.48" width="0" layer="19" extent="1-1"/>
 <wire x1="-78.32" y1="-650.24" x2="-78.32" y2="-655.32" width="0" layer="19" extent="1-1"/>
@@
 <wire x1="-123.19" y1="-735.33" x2="-120.65" y2="-735.33" width="0" layer="19" extent="1-1"/>
 <wire x1="-125.73" y1="-735.33" x2="-123.19" y2="-735.33" width="0" layer="19" extent="1-1"/>
+<wire x1="-129.54" y1="-751.84" x2="-125.73" y2="-735.33" width="0" layer="19" extent="1-1"/>
+<wire x1="-135.89" y1="-751.84" x2="-129.54" y2="-751.84" width="0" layer="19" extent="1-1"/>
+<wire x1="-142.24" y1="-751.84" x2="-135.89" y2="-751.84" width="0" layer="19" extent="1-1"/>
 <wire x1="-16.51" y1="-264.9474" x2="-27.52" y2="-509.27" width="0" layer="19" extent="1-1"/>
 <wire x1="48.57" y1="31.37" x2="-16.51" y2="-264.9474" width="0" layer="19" extent="1-1"/>
@@
 <wire x1="53.07" y1="31.37" x2="-123.9" y2="-748.03" width="0" layer="19" extent="1-1"/>
 </signal>
+<signal name="PA0">
+<contactref element="PORTA" pad="1"/>
+<contactref element="U1" pad="78"/>
+<wire x1="57.07" y1="47.37" x2="-132.08" y2="-741.68" width="0" layer="19" extent="1-1"/>
+</signal>
+<signal name="PA2">
+<contactref element="PORTA" pad="3"/>
+<contactref element="U1" pad="76"/>
+<wire x1="58.07" y1="47.37" x2="-132.08" y2="-744.22" width="0" layer="19" extent="1-1"/>
+</signal>
+<signal name="PA4">
+<contactref element="PORTA" pad="5"/>
+<contactref element="U1" pad="74"/>
+<wire x1="60.07" y1="44.87" x2="-132.08" y2="-746.76" width="0" layer="19" extent="1-1"/>
+</signal>
+<signal name="PA6">
+<contactref element="PORTA" pad="7"/>
+<contactref element="U1" pad="72"/>
+<wire x1="60.07" y1="43.87" x2="-132.08" y2="-749.3" width="0" layer="19" extent="1-1"/>
+</signal>
+<signal name="PA1">
+<contactref element="PORTA" pad="2"/>
+<contactref element="U1" pad="77"/>
+<wire x1="57.57" y1="47.37" x2="-129.54" y2="-741.68" width="0" layer="19" extent="1-1"/>
+</signal>
+<signal name="PA3">
+<contactref element="PORTA" pad="4"/>
+<contactref element="U1" pad="75"/>
+<wire x1="60.07" y1="45.37" x2="-129.54" y2="-744.22" width="0" layer="19" extent="1-1"/>
+</signal>
+<signal name="PA5">
+<contactref element="PORTA" pad="6"/>
+<contactref element="U1" pad="73"/>
+<wire x1="60.07" y1="44.37" x2="-129.54" y2="-746.76" width="0" layer="19" extent="1-1"/>
+</signal>
+<signal name="PA7">
+<contactref element="PORTA" pad="8"/>
+<contactref element="U1" pad="71"/>
+<wire x1="60.07" y1="43.37" x2="-129.54" y2="-749.3" width="0" layer="19" extent="1-1"/>
+</signal>
+<signal name="PE0">
+<contactref element="PORTE" pad="1"/>
+<contactref element="U1" pad="2"/>
+<wire x1="44.07" y1="44.87" x2="-138.43" y2="-741.68" width="0" layer="19" extent="1-1"/>
+</signal>
+<signal name="PE2">
+<contactref element="PORTE" pad="3"/>
+<contactref element="U1" pad="4"/>
+<wire x1="44.07" y1="43.87" x2="-138.43" y2="-744.22" width="0" layer="19" extent="1-1"/>
+</signal>
+<signal name="PE4">
+<contactref element="PORTE" pad="5"/>
+<contactref element="U1" pad="6"/>
+<wire x1="44.07" y1="42.87" x2="-138.43" y2="-746.76" width="0" layer="19" extent="1-1"/>
+</signal>
+<signal name="PE6">
+<contactref element="PORTE" pad="7"/>
+<contactref element="U1" pad="8"/>
+<wire x1="44.07" y1="41.87" x2="-138.43" y2="-749.3" width="0" layer="19" extent="1-1"/>
+</signal>
+<signal name="PE1">
+<contactref element="PORTE" pad="2"/>
+<contactref element="U1" pad="3"/>
+<wire x1="44.07" y1="44.37" x2="-135.89" y2="-741.68" width="0" layer="19" extent="1-1"/>
+</signal>
+<signal name="PE3">
+<contactref element="PORTE" pad="4"/>
+<contactref element="U1" pad="5"/>
+<wire x1="44.07" y1="43.37" x2="-135.89" y2="-744.22" width="0" layer="19" extent="1-1"/>
+</signal>
+<signal name="PE5">
+<contactref element="PORTE" pad="6"/>
+<contactref element="U1" pad="7"/>
+<wire x1="44.07" y1="42.37" x2="-135.89" y2="-746.76" width="0" layer="19" extent="1-1"/>
+</signal>
+<signal name="PE7">
+<contactref element="PORTE" pad="8"/>
+<contactref element="U1" pad="9"/>
+<wire x1="44.07" y1="41.37" x2="-135.89" y2="-749.3" width="0" layer="19" extent="1-1"/>
+</signal>
+<signal name="PF0">
+<contactref element="PORTF" pad="1"/>
+<contactref element="U1" pad="97"/>
+<wire x1="47.57" y1="47.37" x2="-144.78" y2="-741.68" width="0" layer="19" extent="1-1"/>
+</signal>
+<signal name="PF2">
+<contactref element="PORTF" pad="3"/>
+<contactref element="U1" pad="95"/>
+<wire x1="48.57" y1="47.37" x2="-144.78" y2="-744.22" width="0" layer="19" extent="1-1"/>
+</signal>
+<signal name="PF4">
+<contactref element="PORTF" pad="5"/>
+<contactref element="U1" pad="93"/>
+<wire x1="49.57" y1="47.37" x2="-144.78" y2="-746.76" width="0" layer="19" extent="1-1"/>
+</signal>
+<signal name="PF6">
+<contactref element="PORTF" pad="7"/>
+<contactref element="U1" pad="91"/>
+<wire x1="50.57" y1="47.37" x2="-144.78" y2="-749.3" width="0" layer="19" extent="1-1"/>
+</signal>
+<signal name="PF7">
+<contactref element="PORTF" pad="8"/>
+<contactref element="U1" pad="90"/>
+<wire x1="51.07" y1="47.37" x2="-142.24" y2="-749.3" width="0" layer="19" extent="1-1"/>
+</signal>
+<signal name="PF5">
+<contactref element="PORTF" pad="6"/>
+<contactref element="U1" pad="92"/>
+<wire x1="50.07" y1="47.37" x2="-142.24" y2="-746.76" width="0" layer="19" extent="1-1"/>
+</signal>
+<signal name="PF3">
+<contactref element="PORTF" pad="4"/>
+<contactref element="U1" pad="94"/>
+<wire x1="49.07" y1="47.37" x2="-142.24" y2="-744.22" width="0" layer="19" extent="1-1"/>
+</signal>
+<signal name="PF1">
+<contactref element="PORTF" pad="2"/>
+<contactref element="U1" pad="96"/>
+<wire x1="48.07" y1="47.37" x2="-142.24" y2="-741.68" width="0" layer="19" extent="1-1"/>
+</signal>
 </signals>

Commit message: quelques ports
Parts:
- added SV1, SV2, SV3: (no value), con-lstb:MA10-1W
- moved U$2 702.7 mm to (82.5, 14.0)
- moved CBAT 112.8 mm to (57.1, 67.3), turned to 180 degrees
- moved RBAT 102.4 mm to (61.0, 63.5), turned to 180 degrees
- moved RIN 102.4 mm to (53.3, 63.5), turned to 180 degrees
- moved U2 80.3 mm to (55.9, 57.1), turned to 270 degrees
- moved U3 74.1 mm to (80.0, 50.8), turned to 270 degrees
Connections:
- new net N$101: U1.14
- new net N$102: U1.13
- new net N$103: U1.12
- new net N$56: SV1.1
- new net N$57: SV1.2
- new net N$58: SV1.3
- new net N$59: SV1.4
- new net N$60: SV1.5
- new net N$66: SV2.10
- new net N$67: SV2.9
- new net N$68: SV2.8
- new net N$69: SV2.7
- new net N$70: SV2.6
- new net N$71: SV2.5
- new net N$72: SV2.4
- new net N$73: SV2.3
- new net N$74: SV2.2
- new net N$75: SV2.1
- new net N$76: SV3.10
- new net N$77: SV3.9
- new net N$78: SV3.8
- new net N$79: SV3.7
- new net N$80: SV3.6
- new net N$81: SV3.5
- new net N$82: SV3.4
- new net N$83: SV3.3
- new net N$84: SV3.2
- new net N$85: SV3.1
- new net PB4: SV1.7, U1.23
- new net PB5: SV1.8, U1.24
- new net PB6: SV1.9, U1.25
- new net PB7: SV1.10, U1.26
- new net PD3: U1.46
- new net PD4: U1.47
- new net PD5: U1.48
- new net PD6: U1.49
- new net PD7: U1.50
- new net PG0: U1.51
- new net PG1: U1.52
- new net PG2: U1.70
- new net PG3: U1.28
- new net PG4: U1.29
- new net PG5: SV1.6, U1.1

Commit message: J'ai travaillé sur le schematic du PCB. Pas mal final
Parts:
- added C_AREF: 0.1u, SparkFun-Capacitors:0603-CAP
- added J2, J3: FEMALE 2x3, SparkFun-Connectors:2X3
- added J4, J5: (no value), SparkFun-Connectors:1X04_LOCK
- added PORTB, PORTD, PORTG, PORTH, PORTJ, PORTK, PORTL: (no value), SparkFun-Connectors:AVR_ICSP
- added R_MISO_1, R_MISO_2, R_MISO_3, R_MOSI_1, R_MOSI_2, R_MOSI_3, R_RESET_1, R_RESET_2, R_RESET_3, R_SCK_1, R_SCK_2, R_SCK_3: 500, resistor:R0603
- added R_PU_RESET: 4.7k, resistor:R0603
- R_PU_SS: value 1K -> 4.7k
- moved PORTF 230.0 mm to (-151.1, -976.6)
- moved PORTE 202.4 mm to (-151.1, -948.7)
- renumbered RSS to R_PU_SS
Connections:
- net N$14 renamed BAT+
- net N$40 renamed BAT-
- net N$42 renamed SS
- removed net N$101: U1.14
- removed net N$102: U1.13
- removed net N$103: U1.12
- removed net N$31: ICSP.7, U1.21
- removed net PWMH1: ESC1_PWM.1, ESC4_PWM.1, U1.15, U1.18
- removed net PWMH2: ESC3_PWM.1, U1.16
- removed net PWMH3: ESC2_PWM.1, U1.17
- new net CV3P3: PORTG.8
- new net MISO: R_MISO_1.1, R_MISO_2.1, R_MISO_3.1, U1.22
- new net MOSI: R_MOSI_1.1, R_MOSI_2.1, R_MOSI_3.1, U1.21
- new net N$42: J3.3, R_SCK_3.2
- new net N$61: ICSP.5, R_RESET_1.2
- new net N$62: C_AREF.1, U1.98
- new net N$63: J2.5, R_RESET_2.2
- new net N$64: J3.5, R_RESET_3.2
- new net PB0: PORTB.1
- new net PB1: PORTB.2
- new net PB2: PORTB.3
- new net PB3: PORTB.4
- new net PD0: PORTD.1
- new net PD1: PORTD.2
- new net PD2: PORTD.3
- new net PF0_PF2: CREF.1, U1.95, U1.97, U2.17
- new net PH0: PORTH.1, U1.12
- new net PH1: PORTH.2, U1.13
- new net PH2: PORTH.3, U1.14
- new net PH3: PORTH.4, U1.15
- new net PH4: PORTH.5, U1.16
- new net PH5: PORTH.6, U1.17
- new net PH6: PORTH.7, U1.18
- new net PH7: PORTH.8, U1.27
- new net PJ0: PORTJ.1
- new net PJ1: PORTJ.2
- new net PJ2: PORTJ.3
- new net PJ3: PORTJ.4
- new net PJ4: PORTJ.5
- new net PJ5: PORTJ.6
- new net PJ6: PORTJ.7, U1.69
- new net PJ7: PORTJ.8, U1.79
- new net PK0: PORTK.1, U1.89
- new net PK1: PORTK.2, U1.88
- new net PK2: PORTK.3, U1.87
- new net PK3: PORTK.4, U1.86
- new net PK4: PORTK.5, U1.85
- new net PK5: PORTK.6, U1.84
- new net PK6: PORTK.7, U1.83
- new net PK7: PORTK.8, U1.82
- new net PL0: ESC1_PWM.1, PORTL.1, U1.35
- new net PL1: ESC2_PWM.1, PORTL.2, U1.36
- new net PL2: ESC3_PWM.1, PORTL.3, U1.37
- new net PL3: ESC4_PWM.1, PORTL.4, U1.38
- new net PL4: PORTL.5, U1.39
- new net PL5: PORTL.6, U1.40
- new net PL6: PORTL.7, U1.41
- new net PL7: PORTL.8, U1.42
- new net RESET: CRESET.1, D1.C, D2.A, R_PU_RESET.1, R_RESET_1.1, R_RESET_2.1, R_RESET_3.1, R_RESET_SWITCH.1, U1.30
- new net SCK: R_SCK_1.1, R_SCK_2.1, R_SCK_3.1, U1.20
- net GND: now also C_AREF.2, J2.6, J3.6, J4.4, J5.4, LED1.C, LED2.C, LED3.C, PORTB.9, PORTD.9, PORTG.7, PORTG.9, PORTH.9, PORTJ.9, PORTK.9, PORTL.9; no longer R_PU_SS.2
- net N$1: now also ICSP.7, R_SCK_1.2; no longer ICSP.9, U1.22
- net N$2: now also R_MOSI_1.2; no longer U1.20
- net N$20: now also J2.4, R_MOSI_2.2; no longer U1.79, U2.13
- net N$21: now also J2.3, R_SCK_2.2; no longer COUT2.1, U1.88, U2.14
- net N$22: now also J2.1, R_MISO_2.2; no longer COUT.1, U1.87, U2.15
- net N$24: now also J3.4, R_MOSI_3.2; no longer CREF.1, U1.86, U2.17
- net N$3: now also ICSP.9, R_MISO_1.2; no longer CRESET.1, D1.C, D2.A, ICSP.5, R_RESET_SWITCH.1, U1.30
- net N$55: now also J3.1, R_MISO_3.2; no longer SG1.-, U1.40
- net PA0: now also SG1.-
- net PA3: now also PORTD.4
- net PB4: now also PORTB.5
- net PB5: now also PORTB.6
- net PB6: now also PORTB.7
- net PB7: now also PORTB.8
- net PD4: now also PORTD.5
- net PD5: now also PORTD.6
- net PD6: now also PORTD.7
- net PD7: now also PORTD.8
- net PF0: no longer U1.97
- net PF1: now also COUT.1, U2.15
- net PF2: no longer U1.95
- net PF3: now also COUT2.1, U2.14
- net PF4: now also U2.13
- net PG0: now also PORTG.1
- net PG1: now also PORTG.2
- net PG2: now also PORTG.3
- net PG3: now also PORTG.4
- net PG4: now also PORTG.5
- net PG5: now also PORTG.6
- net SCL: now also J4.3, J5.3
- net SDA: now also J4.2, J5.2
- net VCC: now also J3.2, J4.1, J5.1, PORTB.10, PORTD.10, PORTG.10, PORTH.10, PORTJ.10, PORTK.10, PORTL.10, R_PU_RESET.2, R_PU_SS.2
- net V_USB: now also J2.2
