File: eagle/Projects/Sij/Sij.brd (EAGLE design)
At the start: 111.4 x 186.7 mm, 136 parts, among them J2 FEMALE 2x3, J3 FEMALE 2x3, U1 ATMEGA2560AU, U2 BQ76925_PW_20, U3 LM1085_KTT_3, U4 LM7805, U5 TC7SU04F

Commit message: joué un peu avec le layout
Parts:
- removed ICSP: (no value), SparkFun-Connectors:AVR_ICSP
- removed J1: (no value), SparkFun-Connectors:1X06_FEMALE_LOCK.010
- removed J2, J3: FEMALE 2x3, SparkFun-Connectors:2X3
- removed J4, J5: (no value), SparkFun-Connectors:1X04_LOCK
- removed JP1, JP2, JP3: (no value), SparkFun-Retired:1X02
- removed SV1, SV2, SV3: (no value), con-lstb:MA10-1W
- removed U$2: M06_IMU, custom_parts:1X06_LONGPADS
- added EXTRA_5V, PROGRAMMER6, SPI: FEMALE 2x3, SparkFun-Connectors:2X3
- added I2C_1, I2C_2: (no value), SparkFun-Connectors:1X04_LOCK
- added IMU: M06_IMU, custom_parts:1X06_LONGPADS
- added JP4CELL, JP5CELL, JP6CELL: (no value), SparkFun-Retired:1X02
- added PROGRAMMER10: (no value), SparkFun-Connectors:AVR_ICSP
- moved PORTK 1088.7 mm to (72.4, 76.2), turned to 90 degrees
- moved PORTJ 1071.4 mm to (95.2, 52.1)
- moved PORTF 1067.9 mm to (27.9, 76.2), turned to 270 degrees
- moved PORTE 1038.1 mm to (14.0, 76.2), turned to 270 degrees
- moved PORTH 1037.4 mm to (5.08, 50.8)
- moved PORTG 1006.2 mm to (81.3, 3.81), turned to 270 degrees
- moved PORTD 993.7 mm to (95.2, 27.9)
- moved PORTL 982.8 mm to (20.3, 5.08), turned to 90 degrees
- moved R_RESET_1 967.7 mm to (43.2, 71.1), turned to 90 degrees
- moved R_RESET_3 961.7 mm to (92.7, 43.2)
- moved PORTB 947.7 mm to (5.08, 27.9)
- moved R_SCK_3 945.9 mm to (97.8, 40.6)
- moved R_MOSI_3 939.7 mm to (92.7, 40.6)
- moved R_RESET_2 939.0 mm to (10.2, 43.2)
- moved R_MISO_3 938.6 mm to (97.8, 43.2)
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Connections:
- removed net N$56: SV1.1
- removed net N$57: SV1.2
- removed net N$58: SV1.3
- removed net N$59: SV1.4
- removed net N$60: SV1.5
- removed net N$66: SV2.10
- removed net N$67: SV2.9
- removed net N$68: SV2.8
- removed net N$69: SV2.7
- removed net N$70: SV2.6
- removed net N$71: SV2.5
- removed net N$72: SV2.4
- removed net N$73: SV2.3
- removed net N$74: SV2.2
- removed net N$75: SV2.1
- removed net N$76: SV3.10
- removed net N$77: SV3.9
- removed net N$78: SV3.8
- removed net N$79: SV3.7
- removed net N$80: SV3.6
- removed net N$81: SV3.5
- removed net N$82: SV3.4
- removed net N$83: SV3.3
- removed net N$84: SV3.2
- removed net N$85: SV3.1
- net GND: now also EXTRA_5V.2, EXTRA_5V.4, EXTRA_5V.6, I2C_1.4, I2C_2.4, IMU.1, IMU.5, PROGRAMMER10.10, PROGRAMMER10.4, PROGRAMMER10.6, PROGRAMMER10.8, PROGRAMMER6.6, SPI.6; no longer ICSP.10, ICSP.4, ICSP.6, ICSP.8, J2.6, J3.6, J4.4, J5.4, U$2.1, U$2.5
- net INT_IMU: now also IMU.2; no longer U$2.2
- net N$1: now also PROGRAMMER10.7; no longer ICSP.7
- net N$2: now also PROGRAMMER10.1; no longer ICSP.1
- net N$20: now also PROGRAMMER6.4; no longer J2.4
- net N$21: now also PROGRAMMER6.3; no longer J2.3
- net N$22: now also PROGRAMMER6.1; no longer J2.1
- net N$24: now also SPI.4; no longer J3.4
- net N$28: now also JP4CELL.1; no longer JP3.1
- net N$29: now also JP4CELL.2, JP5CELL.1; no longer JP2.1, JP3.2
- net N$3: now also PROGRAMMER10.9; no longer ICSP.9
- net N$30: now also JP5CELL.2, JP6CELL.1; no longer JP1.1, JP2.2
- net N$32: now also EXTRA_5V.1, EXTRA_5V.3, EXTRA_5V.5; no longer J1.1, J1.2, J1.3, J1.4, J1.5, J1.6
- net N$42: now also SPI.3; no longer J3.3
- net N$55: now also SPI.1; no longer J3.1
- net N$61: now also PROGRAMMER10.5; no longer ICSP.5
- net N$63: now also PROGRAMMER6.5; no longer J2.5
- net N$64: now also SPI.5; no longer J3.5
- net PB4: no longer SV1.7
- net PB5: no longer SV1.8
- net PB6: no longer SV1.9
- net PB7: no longer SV1.10
- net PG5: no longer SV1.6
- net SCL: now also I2C_1.3, I2C_2.3, IMU.3; no longer J4.3, J5.3, U$2.3
- net SDA: now also I2C_1.2, I2C_2.2, IMU.4; no longer J4.2, J5.2, U$2.4
- net VCC: now also I2C_1.1, I2C_2.1, IMU.6, SPI.2; no longer J3.2, J4.1, J5.1, U$2.6
- net V_BATT: now also JP6CELL.2; no longer JP1.2
- net V_USB: now also PROGRAMMER10.2, PROGRAMMER6.2; no longer ICSP.2, J2.2
Other:
- board size 111.4 x 186.7 mm -> 100 x 80 mm

Commit message: fichiers pour code ESC créés
Connections:
- net PH3: now also ESC1_PWM.1
- net PH4: now also ESC2_PWM.1
- net PL0: no longer ESC1_PWM.1
- net PL1: no longer ESC2_PWM.1
- net PL2: no longer ESC3_PWM.1
- net PL3: now also ESC3_PWM.1; no longer ESC4_PWM.1
- net PL4: now also ESC4_PWM.1
Changed lines of the file:
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@@
 <contactref element="U1" pad="40"/>
 <contactref element="PORTL" pad="6"/>
-<wire x1="50.53" y1="47.88" x2="20.32" y2="6.35" width="0" layer="19" extent="1-1"/>
+<wire x1="20.32" y1="6.35" x2="50.53" y2="47.88" width="0" layer="19" extent="1-1"/>
 </signal>
 <signal name="PL4">
 <contactref element="U1" pad="39"/>
 <contactref element="PORTL" pad="5"/>
-<wire x1="50.03" y1="47.88" x2="20.32" y2="3.81" width="0" layer="19" extent="1-1"/>
+<contactref element="ESC4_PWM" pad="1"/>
+<wire x1="20.32" y1="3.81" x2="50.03" y2="47.88" width="0" layer="19" extent="1-1"/>
+<wire x1="3.81" y1="11.43" x2="20.32" y2="3.81" width="0" layer="19" extent="1-1"/>
 </signal>
 <signal name="PL3">
 <contactref element="U1" pad="38"/>
-<contactref element="ESC4_PWM" pad="1"/>
 <contactref element="PORTL" pad="4"/>
-<wire x1="49.53" y1="47.88" x2="3.81" y2="11.43" width="0" layer="19" extent="1-1"/>
-<wire x1="17.78" y1="6.35" x2="3.81" y2="11.43" width="0" layer="19" extent="1-1"/>
+<contactref element="ESC3_PWM" pad="1"/>
+<wire x1="49.53" y1="47.88" x2="96.52" y2="8.89" width="0" layer="19" extent="1-1"/>
+<wire x1="17.78" y1="6.35" x2="49.53" y2="47.88" width="0" layer="19" extent="1-1"/>
 </signal>
 <signal name="PL2">
 <contactref element="U1" pad="37"/>
-<contactref element="ESC3_PWM" pad="1"/>
 <contactref element="PORTL" pad="3"/>
-<wire x1="96.52" y1="8.89" x2="17.78" y2="3.81" width="0" layer="19" extent="1-1"/>
-<wire x1="49.03" y1="47.88" x2="96.52" y2="8.89" width="0" layer="19" extent="1-1"/>
+<wire x1="17.78" y1="3.81" x2="49.03" y2="47.88" width="0" layer="19" extent="1-1"/>
 </signal>
 <signal name="PL1">
 <contactref element="U1" pad="36"/>
-<contactref element="ESC2_PWM" pad="1"/>
 <contactref element="PORTL" pad="2"/>
-<wire x1="96.52" y1="68.58" x2="15.24" y2="6.35" width="0" layer="19" extent="1-1"/>
-<wire x1="48.53" y1="47.88" x2="96.52" y2="68.58" width="0" layer="19" extent="1-1"/>
+<wire x1="15.24" y1="6.35" x2="48.53" y2="47.88" width="0" layer="19" extent="1-1"/>
 </signal>
 <signal name="PL0">
 <contactref element="U1" pad="35"/>
-<contactref element="ESC1_PWM" pad="1"/>
 <contactref element="PORTL" pad="1"/>
-<wire x1="3.81" y1="68.58" x2="15.24" y2="3.81" width="0" layer="19" extent="1-1"/>
-<wire x1="48.03" y1="47.88" x2="3.81" y2="68.58" width="0" layer="19" extent="1-1"/>
+<wire x1="15.24" y1="3.81" x2="48.03" y2="47.88" width="0" layer="19" extent="1-1"/>
 </signal>
 <signal name="PK7">
@@
 <contactref element="U1" pad="16"/>
 <contactref element="PORTH" pad="5"/>
-<wire x1="41.53" y1="54.38" x2="3.81" y2="50.8" width="0" layer="19" extent="1-1"/>
+<contactref element="ESC2_PWM" pad="1"/>
+<wire x1="41.53" y1="54.38" x2="96.52" y2="68.58" width="0" layer="19" extent="1-1"/>
+<wire x1="3.81" y1="50.8" x2="41.53" y2="54.38" width="0" layer="19" extent="1-1"/>
 </signal>
 <signal name="PH3">
 <contactref element="U1" pad="15"/>
 <contactref element="PORTH" pad="4"/>
-<wire x1="41.53" y1="54.88" x2="6.35" y2="53.34" width="0" layer="19" extent="1-1"/>
+<contactref element="ESC1_PWM" pad="1"/>
+<wire x1="6.35" y1="53.34" x2="41.53" y2="54.88" width="0" layer="19" extent="1-1"/>
+<wire x1="3.81" y1="68.58" x2="6.35" y2="53.34" width="0" layer="19" extent="1-1"/>
 </signal>
 <signal name="PF0_PF2">
