File: eagle/Projects/Sij/Sij.sch (EAGLE design)
At the start: 111 parts, among them U1 ATMEGA2560AU, U2 BQ76925_PW_20, U3 LM1085_KTT_3, U4 LM7805, U5 TC7SU04F

Commit message: J'ai travaillé sur le schematic du PCB. Pas mal final
Parts:
- removed RSS: 1K, resistor:R-US_R0603
- added C_AREF: 0.1u, SparkFun-Capacitors:CAP0603-CAP
- added J2, J3: FEMALE 2x3, SparkFun-Connectors:M03X2FEMALE
- added J4, J5: (no value), SparkFun-Connectors:M04LOCK
- added PORTB, PORTD, PORTG, PORTH, PORTJ, PORTK, PORTL: (no value), SparkFun-Connectors:M05X2PTH
- added R_MISO_1, R_MISO_2, R_MISO_3, R_MOSI_1, R_MOSI_2, R_MOSI_3, R_RESET_1, R_RESET_2, R_RESET_3, R_SCK_1, R_SCK_2, R_SCK_3: 500, resistor:R-US_R0603
- added R_PU_RESET, R_PU_SS: 4.7k, resistor:R-US_R0603
Connections:
- net N$14 renamed BAT+
- net N$40 renamed BAT-
- removed net N$101: U1.PH2(XCK2)
- removed net N$102: U1.PH1(TXD2)
- removed net N$103: U1.PH0(RXD2)
- removed net N$31: ICSP.7, U1.(MOSI/PCINT2)PB2
- removed net PWMH1: ESC1_PWM.1, ESC4_PWM.1, U1.PH3(OC4A), U1.PH6(OC2B)
- removed net PWMH2: ESC3_PWM.1, U1.PH4(OC4B)
- removed net PWMH3: ESC2_PWM.1, U1.PH5(OC4C)
- new net CV3P3: PORTG.8
- new net MISO: R_MISO_1.1, R_MISO_2.1, R_MISO_3.1, U1.(MISO/PCINT3)PB3
- new net MOSI: R_MOSI_1.1, R_MOSI_2.1, R_MOSI_3.1, U1.(MOSI/PCINT2)PB2
- new net N$61: ICSP.5, R_RESET_1.2
- new net N$62: C_AREF.1, U1.AREF
- new net N$63: J2.5, R_RESET_2.2
- new net N$64: J3.5, R_RESET_3.2
- new net PB0: PORTB.1
- new net PB1: PORTB.2
- new net PB2: PORTB.3
- new net PB3: PORTB.4
- new net PD0: PORTD.1
- new net PD1: PORTD.2
- new net PD2: PORTD.3
- new net PF0_PF2: CREF.1, U1.(ADC0)PF0, U1.(ADC2)PF2, U2.VREF
- new net PH0: PORTH.1, U1.PH0(RXD2)
- new net PH1: PORTH.2, U1.PH1(TXD2)
- new net PH2: PORTH.3, U1.PH2(XCK2)
- new net PH3: PORTH.4, U1.PH3(OC4A)
- new net PH4: PORTH.5, U1.PH4(OC4B)
- new net PH5: PORTH.6, U1.PH5(OC4C)
- new net PH6: PORTH.7, U1.PH6(OC2B)
- new net PH7: PORTH.8, U1.PH7(T4)
- new net PJ0: PORTJ.1
- new net PJ1: PORTJ.2
- new net PJ2: PORTJ.3
- new net PJ3: PORTJ.4
- new net PJ4: PORTJ.5
- new net PJ5: PORTJ.6
- new net PJ6: PORTJ.7, U1.PJ6(PCINT15)
- new net PJ7: PORTJ.8, U1.PJ7
- new net PK0: PORTK.1, U1.PK0(ADC8/PCINT16)
- new net PK1: PORTK.2, U1.PK1(ADC9/PCINT17)
- new net PK2: PORTK.3, U1.PK2(ADC10/PCINT18)
- new net PK3: PORTK.4, U1.PK3(ADC11/PCINT19)
- new net PK4: PORTK.5, U1.PK4(ADC12/PCINT20)
- new net PK5: PORTK.6, U1.PK5(ADC13/PCINT21)
- new net PK6: PORTK.7, U1.PK6(ADC14/PCINT22)
- new net PK7: PORTK.8, U1.PK7(ADC15/PCINT23)
- new net PL0: ESC1_PWM.1, PORTL.1, U1.PL0(ICP4)
- new net PL1: ESC2_PWM.1, PORTL.2, U1.PL1(ICP5)
- new net PL2: ESC3_PWM.1, PORTL.3, U1.PL2(T5)
- new net PL3: ESC4_PWM.1, PORTL.4, U1.PL3(OC5A)
- new net PL4: PORTL.5, U1.PL4(OC5B)
- new net PL5: PORTL.6, U1.PL5(OC5C)
- new net PL6: PORTL.7, U1.PL6
- new net PL7: PORTL.8, U1.PL7
- new net RESET: CRESET.1, D1.C, D2.A, R_PU_RESET.1, R_RESET_1.1, R_RESET_2.1, R_RESET_3.1, R_RESET_SWITCH.1, U1.RESET
- new net SCK: R_SCK_1.1, R_SCK_2.1, R_SCK_3.1, U1.(SCK/PCINT1)PB1
- new net SS: R_PU_SS.1, U1.(SS/PCINT0)PB0
- net GND: now also C_AREF.2, J2.6, J3.6, J4.4, J5.4, LED1.C, LED2.C, LED3.C, PORTB.9, PORTD.9, PORTG.7, PORTG.9, PORTH.9, PORTJ.9, PORTK.9, PORTL.9; no longer RSS.2
- net N$1: now also ICSP.7, R_SCK_1.2; no longer ICSP.9, U1.(MISO/PCINT3)PB3
- net N$2: now also R_MOSI_1.2; no longer U1.(SCK/PCINT1)PB1
- net N$20: now also J2.4, R_MOSI_2.2; no longer U1.PJ7, U2.ALERT
- net N$21: now also J2.3, R_SCK_2.2; no longer COUT2.1, U1.PK1(ADC9/PCINT17), U2.VIOUT
- net N$22: now also J2.1, R_MISO_2.2; no longer COUT.1, U1.PK2(ADC10/PCINT18), U2.VCOUT
- net N$24: now also J3.4, R_MOSI_3.2; no longer CREF.1, U1.PK3(ADC11/PCINT19), U2.VREF
- net N$3: now also ICSP.9, R_MISO_1.2; no longer CRESET.1, D1.C, D2.A, ICSP.5, R_RESET_SWITCH.1, U1.RESET
- net N$42: now also J3.3, R_SCK_3.2; no longer RSS.1, U1.(SS/PCINT0)PB0
- net N$55: now also J3.1, R_MISO_3.2; no longer SG1.2, U1.PL5(OC5C)
- net PA0: now also SG1.2
- net PA3: now also PORTD.4
- net PB4: now also PORTB.5
- net PB5: now also PORTB.6
- net PB6: now also PORTB.7
- net PB7: now also PORTB.8
- net PD4: now also PORTD.5
- net PD5: now also PORTD.6
- net PD6: now also PORTD.7
- net PD7: now also PORTD.8
- net PF0: no longer U1.(ADC0)PF0
- net PF1: now also COUT.1, U2.VCOUT
- net PF2: no longer U1.(ADC2)PF2
- net PF3: now also COUT2.1, U2.VIOUT
- net PF4: now also U2.ALERT
- net PG0: now also PORTG.1
- net PG1: now also PORTG.2
- net PG2: now also PORTG.3
- net PG3: now also PORTG.4
- net PG4: now also PORTG.5
- net PG5: now also PORTG.6
- net SCL: now also J4.3, J5.3
- net SDA: now also J4.2, J5.2
- net VCC: now also J3.2, J4.1, J5.1, PORTB.10, PORTD.10, PORTG.10, PORTH.10, PORTJ.10, PORTK.10, PORTL.10, R_PU_RESET.2, R_PU_SS.2
- net V_USB: now also J2.2
Other:
- note added: "5V main"
- note added: "External I2C 1"
- note added: "External I2C 2"
- note added: "External SPI"
- note added: "Extra 5V high power"
- note added: "Input Power Selector"
- note added: "Ports"
- note added: "Programmer 10 pin"
- note added: "Programmer 6 pin"
- note removed: "Programmer"
- note removed: "To ADC ref voltage"
- moved on the sheet: BAT+, BAT-, CBAT, CIN, CIN1, CIN2, CIN3, CIN4, CIN5, CIN6, CIN_1085, CIN_7805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

Commit message: joué un peu avec le layout
Parts:
- removed J1: (no value), SparkFun-Connectors:M06FEMALE_LOCK
- removed SV1, SV2, SV3: (no value), con-lstb:MA10-1W
- added EXTRA_5V: FEMALE 2x3, SparkFun-Connectors:M03X2FEMALE
- renumbered ICSP to PROGRAMMER10, J2 to PROGRAMMER6, J3 to SPI, J4 to I2C_1, J5 to I2C_2, JP1 to JP6CELL, JP2 to JP5CELL, JP3 to JP4CELL, U$2 to IMU
Connections:
- removed net N$56: SV1.1
- removed net N$57: SV1.2
- removed net N$58: SV1.3
- removed net N$59: SV1.4
- removed net N$60: SV1.5
- removed net N$66: SV2.10
- removed net N$67: SV2.9
- removed net N$68: SV2.8
- removed net N$69: SV2.7
- removed net N$70: SV2.6
- removed net N$71: SV2.5
- removed net N$72: SV2.4
- removed net N$73: SV2.3
- removed net N$74: SV2.2
- removed net N$75: SV2.1
- removed net N$76: SV3.10
- removed net N$77: SV3.9
- removed net N$78: SV3.8
- removed net N$79: SV3.7
- removed net N$80: SV3.6
- removed net N$81: SV3.5
- removed net N$82: SV3.4
- removed net N$83: SV3.3
- removed net N$84: SV3.2
- removed net N$85: SV3.1
- net GND: now also EXTRA_5V.2, EXTRA_5V.4, EXTRA_5V.6
- net N$32: now also EXTRA_5V.1, EXTRA_5V.3, EXTRA_5V.5; no longer J1.1, J1.2, J1.3, J1.4, J1.5, J1.6
- net PB4: no longer SV1.7
- net PB5: no longer SV1.8
- net PB6: no longer SV1.9
- net PB7: no longer SV1.10
- net PG5: no longer SV1.6

Commit message: fichiers pour code ESC créés
Connections:
- net PH3: now also ESC1_PWM.1
- net PH4: now also ESC2_PWM.1
- net PL0: no longer ESC1_PWM.1
- net PL1: no longer ESC2_PWM.1
- net PL2: no longer ESC3_PWM.1
- net PL3: now also ESC3_PWM.1; no longer ESC4_PWM.1
- net PL4: now also ESC4_PWM.1
