File: eagle/Projects/Sij/Sij.sch (EAGLE design)
At the start: 133 parts, among them U1 ATMEGA2560AU, U2 BQ76925_PW_20, U3 LM1085_KTT_3, U4 LM7805, U5 TC7SU04F

Commit message: Modifié le PCB
Parts:
- removed ESC1+, ESC1-, ESC2+, ESC2-, ESC3+, ESC3-, ESC4+, ESC4-: BULLET_PAD, custom_parts:BULLET_PAD
- removed ESC1_PWM, ESC3_PWM, ESC4_PWM: 640455 TE connectivity, SparkFun-Connectors:M02PTH
- removed ESC2_PWM: (no value), SparkFun-Connectors:M02PTH
- removed I2C_2: (no value), SparkFun-Connectors:M04LOCK
- removed J_RECEIVER_GND, J_RECEIVER_SIG, J_RECEIVER_VCC: (no value), SparkFun-Connectors:M07
- removed PROGRAMMER6: FEMALE 2x3, SparkFun-Connectors:M03X2FEMALE
- removed R_MISO_2, R_MOSI_2, R_RESET_2, R_SCK_2: 500, resistor:R-US_R0603
- added ESC_BL+, ESC_BL-, ESC_BR+, ESC_BR-, ESC_FL+, ESC_FL-, ESC_FR+, ESC_FR-: BULLET_PAD, custom_parts:BULLET_PAD
- added ESC_BL_PWM, ESC_BR_PWM, ESC_FL_PWM, ESC_FR_PWM: 640455 TE connectivity, SparkFun-Connectors:M02PTH
- added LCD_VD1, LCD_VD2: (no value), resistor:R-US_R0603
- added U$2: RF_CONTROL_3X7_CON, custom_parts:RF_CONTROL_3X7_CON
Connections:
- removed net N$20: PROGRAMMER6.4, R_MOSI_2.2
- removed net N$21: PROGRAMMER6.3, R_SCK_2.2
- removed net N$22: PROGRAMMER6.1, R_MISO_2.2
- removed net N$63: PROGRAMMER6.5, R_RESET_2.2
- removed net PJ0: PORTJ.1
- removed net PJ1: PORTJ.2
- removed net PJ2: PORTJ.3
- removed net PJ3: PORTJ.4
- removed net PJ4: PORTJ.5
- removed net PJ5: PORTJ.6
- new net LCD_V0: LCD_VD1.1, LCD_VD2.2, PORTA.10
- net BAT+: now also ESC_BL+.PAD, ESC_BR+.PAD, ESC_FL+.PAD, ESC_FR+.PAD; no longer ESC1+.PAD, ESC2+.PAD, ESC3+.PAD, ESC4+.PAD
- net CH1: now also PORTJ.1, U$2.1; no longer J_RECEIVER_SIG.1
- net CH2: now also PORTJ.2, U$2.2; no longer J_RECEIVER_SIG.2
- net CH3: now also PORTJ.3, U$2.3; no longer J_RECEIVER_SIG.3
- net CH4: now also PORTJ.4, U$2.4; no longer J_RECEIVER_SIG.4
- net CH5: now also PORTJ.5, U$2.5; no longer J_RECEIVER_SIG.5
- net CH6: now also PORTJ.6, U$2.6; no longer J_RECEIVER_SIG.6
- net GND: now also ESC_BL_PWM.2, ESC_BR_PWM.2, ESC_FL_PWM.2, ESC_FR_PWM.2, LCD_VD2.1, U$2.GND; no longer ESC1_PWM.2, ESC2_PWM.2, ESC3_PWM.2, ESC4_PWM.2, I2C_2.4, J_RECEIVER_GND.1, J_RECEIVER_GND.2, J_RECEIVER_GND.3, J_RECEIVER_GND.4, J_RECEIVER_GND.5, J_RECEIVER_GND.6, PROGRAMMER6.6
- net GND-ISO: now also ESC_BL-.PAD, ESC_BR-.PAD, ESC_FL-.PAD, ESC_FR-.PAD; no longer ESC1-.PAD, ESC2-.PAD, ESC3-.PAD, ESC4-.PAD
- net MISO: no longer R_MISO_2.1
- net MOSI: no longer R_MOSI_2.1
- net PH3: now also ESC_BL_PWM.1; no longer ESC1_PWM.1
- net PH4: now also ESC_FL_PWM.1; no longer ESC2_PWM.1
- net PL3: now also ESC_FR_PWM.1; no longer ESC3_PWM.1
- net PL4: now also ESC_BR_PWM.1; no longer ESC4_PWM.1
- net RESET: no longer R_RESET_2.1
- net SCK: no longer R_SCK_2.1
- net SCL: no longer I2C_2.3
- net SDA: no longer I2C_2.2
- net VCC: now also LCD_VD1.2, U$2.5V; no longer I2C_2.1, J_RECEIVER_VCC.1, J_RECEIVER_VCC.2, J_RECEIVER_VCC.3, J_RECEIVER_VCC.4, J_RECEIVER_VCC.5, J_RECEIVER_VCC.6, PORTA.10
- net V_USB: no longer PROGRAMMER6.2
Other:
- note added: "Buzzer"
- note added: "External I2C"
- note added: "LCD contrast"
- note removed: "5V USB"
- note removed: "External I2C 1"
- note removed: "External I2C 2"
- note removed: "Programmer 6 pin"
- moved on the sheet: BAT+, BAT-, CBAT, CIN, CIN1, CIN2, CIN3, CIN4, CIN5, CIN6, CIN_1085, CIN_7805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

Commit message: presque terminé le layout. Après genre 20h de travail acharné!
Parts:
- removed I2C_1: (no value), SparkFun-Connectors:M04LOCK
- removed LED10, LED11, LED8, LED9: (no value), led:LEDCHIPLED_0805
- removed RLED10, RLED11, RLED8, RLED9: 91, resistor:R-US_R0603
- added BAT, LED0, USB, VCC: (no value), led:LEDCHIPLED_0805
- added I2C: (no value), SparkFun-Connectors:M041X04_NO_SILK
- added RLED0, R_BAT, R_USB, R_VCC: (no value), resistor:R-US_R0603
- C_CRY1, C_CRY2: value 20pF -> 22pF
- RLED1, RLED3, RLED4, RLED5, RLED6, RLED7: value 56 -> (none)
- RLED2: value 316 -> (none)
- R_LCD1: value (none) -> 2k
- R_LCD2: value (none) -> 330
- renumbered BAT+ to BAT_IN+, BAT- to BAT_IN-, CIN_1085 to CI_10, CIN_7805 to CI_78, COUT_1085 to CO_10, COUT_7805 to CO_78, CRESET to C_RES, CRYSTAL to 16MHZ, C_CRYSTAL_1 to C_CRY1, C_CRYSTAL_2 to C_CRY2, C_DECOUPLING1 to C_DECO1, C_DECOUPLING2 to C_DECO2, C_DECOUPLING3 to C_DECO3, C_DECOUPLING4 to C_DECO4, D1 to D_PD_RES, D2 to D_PU_RES, D_POWER_SEL to D_SEL, ESC_BL+ to BAT+3, ESC_BL- to BAT-4, ESC_BL_PWM to ESC_BL, ESC_BR+ to BAT+2, ESC_BR- to BAT-1, ESC_BR_PWM to ESC_BR, ESC_FL+ to BAT+4, ESC_FL- to BAT-2, ESC_FL_PWM to ESC_FL, ESC_FR+ to BAT+1, ESC_FR- to BAT-3, ESC_FR_PWM to ESC_FR, IMU to IMU_BOARD, JP4CELL to JP4, JP5CELL to JP5, JP6CELL to JP6, LCD_VD1 to R_LCD1, LCD_VD2 to R_LCD2, Q_POWER_SEL1 to Q_SEL1, Q_POWER_SEL2 to Q_SEL2, R2 to R2_10, RESET_SWITCH to RES_SW, R_1085 to R_10, R_MISO_1 to RSPI4, R_MISO_3 to RSPI5, R_MOSI_1 to RSPI1, R_MOSI_3 to RSPI8, R_PULL_DOWN_POWER_SEL to R_PD_SEL, R_PULL_UP_POWER_SEL to R_PU_SEL, R_PU_RESET to R_PU_RES, R_RESET_1 to RSPI2, R_RESET_3 to RSPI7, R_RESET_SWITCH to R_RES, R_SCK_1 to RSPI3, R_SCK_3 to RSPI6, SG1 to BUZZ, U$1 to BAT-MONIT, U$2 to RADIO_CONTROLLER, U$3 to POWER_SWITCH, U1 to ATMEGA2560, U2 to BQ76925, U3 to LM1085, U4 to LM7805, U5 to INV
Connections:
- removed net N$49: ATMEGA2560.(A13)PC5, RLED6.1
- removed net N$50: ATMEGA2560.(A12)PC4, RLED7.1
- removed net N$51: ATMEGA2560.(A11)PC3, RLED8.1
- removed net N$52: ATMEGA2560.(A10)PC2, RLED9.1
- removed net N$53: ATMEGA2560.(A9)PC1, RLED10.1
- removed net N$54: ATMEGA2560.(A8)PC0, RLED11.1
- removed net PB0: PORTB.1
- removed net PB1: PORTB.2
- removed net PB2: PORTB.3
- removed net PB3: PORTB.4
- removed net PD0: PORTD.1
- removed net PD1: PORTD.2
- removed net PD2: PORTD.3
- removed net PF0: PORTF.1
- removed net PF0_PF2: ATMEGA2560.(ADC0)PF0, ATMEGA2560.(ADC2)PF2, BQ76925.VREF, CREF.1
- removed net PF2: PORTF.3
- removed net RLED2: LED2.A, RLED2.2
- new net N$14: ATMEGA2560.(A15)PC7, LED7.A
- new net N$20: ATMEGA2560.(A13)PC5, LED5.A
- new net N$21: ATMEGA2560.(A12)PC4, LED4.A
- new net N$22: ATMEGA2560.(A11)PC3, LED3.A
- new net N$31: ATMEGA2560.(A8)PC0, LED0.A
- new net N$40: LED6.C, RLED6.1
- new net PF0_2: ATMEGA2560.(ADC0)PF0, ATMEGA2560.(ADC2)PF2, BQ76925.VREF, CREF.1, PORTF.1, PORTF.3
- net BAT+: now also BAT.A; no longer RLED2.1
- net CH1: now also ATMEGA2560.PJ5(PCINT14); no longer ATMEGA2560.PJ0(RXD3/PCINT9)
- net CH2: now also ATMEGA2560.PJ4(PCINT13); no longer ATMEGA2560.PJ1(TXD3/PCINT10)
- net CH3: now also ATMEGA2560.PJ3(PCINT12); no longer ATMEGA2560.PJ2(XCK3/PCINT11)
- net CH4: now also ATMEGA2560.PJ2(XCK3/PCINT11); no longer ATMEGA2560.PJ3(PCINT12)
- net CH5: now also ATMEGA2560.PJ1(TXD3/PCINT10); no longer ATMEGA2560.PJ4(PCINT13)
- net CH6: now also ATMEGA2560.PJ0(RXD3/PCINT9); no longer ATMEGA2560.PJ5(PCINT14)
- net CV3P3: now also BQ76925.V3P3, CV3P3.1
- net GND: now also I2C.4, RLED0.2, RLED1.2, RLED2.2, RLED3.2, RLED4.2, RLED5.2, RLED6.2, RLED7.2, R_BAT.2, R_USB.2, R_VCC.2; no longer I2C_1.4, LED1.C, LED10.C, LED11.C, LED2.C, LED3.C, LED4.C, LED5.C, LED6.C, LED7.C, LED8.C, LED9.C
- net INT_IMU: now also PORTD.3
- net MISO: now also PORTB.4
- net MOSI: now also PORTB.3
- net N$19: now also ATMEGA2560.(A14)PC6, LED6.A; no longer LED4.A, RLED4.2
- net N$25: now also ATMEGA2560.(A10)PC2, LED2.A; no longer LED5.A, RLED5.2
- net N$26: now also ATMEGA2560.(A9)PC1, LED1.A; no longer BQ76925.V3P3, CV3P3.1
- net N$35: now also R_USB.1, USB.C; no longer LED1.A, RLED1.2
- net N$38: now also R_VCC.1, VCC.C; no longer LED3.A, RLED3.2
- net N$39: now also LED7.C, RLED7.1; no longer LED6.A, RLED6.2
- net N$41: now also LED5.C, RLED5.1; no longer LED7.A, RLED7.2
- net N$43: now also LED4.C, RLED4.1; no longer LED8.A, RLED8.2
- net N$44: now also LED3.C, RLED3.1; no longer LED9.A, RLED9.2
- net N$45: now also LED2.C, RLED2.1; no longer LED10.A, RLED10.2
- net N$46: now also LED1.C, RLED1.1; no longer LED11.A, RLED11.2
- net N$47: now also LED0.C, RLED0.1; no longer ATMEGA2560.(A15)PC7, RLED4.1
- net N$48: now also BAT.C, R_BAT.1; no longer ATMEGA2560.(A14)PC6, RLED5.1
- net PA3: no longer PORTD.4
- net PD3: now also PORTD.4
- net SCK: now also PORTB.2
- net SCL: now also I2C.3, PORTD.1; no longer I2C_1.3
- net SDA: now also I2C.2, PORTD.2; no longer I2C_1.2
- net SS: now also PORTB.1
- net VCC: now also I2C.1, VCC.A; no longer I2C_1.1, RLED1.1, SPI.2
- net V_USB: now also SPI.2, USB.A; no longer RLED3.1
Other:
- moved on the sheet: LED1, LED2, LED3, LED4, LED5, LED6, LED7, RLED1, RLED2, RLED3, RLED4, RLED5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
